File: pcb/v1/atreyu-pcb2.kicad_sch (KiCad schematic)
At the start: 126 parts, among them SW1 SW_Push, SW2 RotaryEncoder_Switch, SW3 RotaryEncoder_Switch, U1 Elite-C

Commit message: Added top and bottom pictures for v1, and other small changes.
Parts:
- D1, D10, D11, D12, D13, D14, D15, D16, D17, D18, D19, D2, D20, D21, D22, D23, D24, D25, D26, D27, D28, D29, D3, D30, D31, D32, D33, D34, D35, D36, D37, D38, D39, D4, D40, D41, D42, D43, D44, D45, D46, D47, D48, D49, D5, D50, D51, D52, D53, D54, D55, D56, D57, D58, D59, D6, D60, D7, D8, D9: footprint footprints:D3_hybrid_common_hole -> footprints:D3_hybrid_common_hole_connected_fix
- SW1: footprint footprints:ResetSW_1side -> footprints:SW_Tactile_SPST_Angled_MJTP1117

Commit message: Fixed reset button, take 2.
Parts:
- SW1: footprint footprints:SW_Tactile_SPST_Angled_MJTP1117 -> footprints:SW_Tactile_SPST_Angled_MJTP1117_fixed
Changed lines of the file:
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@@
     (property "Reference" "SW1" (id 0) (at 146.05 146.431 0))
     (property "Value" "SW_Push" (id 1) (at 146.05 148.7424 0))
-    (property "Footprint" "footprints:SW_Tactile_SPST_Angled_MJTP1117" (id 2) (at 146.05 148.59 0)
+    (property "Footprint" "footprints:SW_Tactile_SPST_Angled_MJTP1117_fixed" (id 2) (at 146.05 148.59 0)
       (effects (font (size 1.27 1.27)) hide)
     )
@@
     )
     (path "/f228d0b8-6193-4b01-bde8-b5aa48a06a4d"
-      (reference "SW1") (unit 1) (value "SW_Push") (footprint "footprints:SW_Tactile_SPST_Angled_MJTP1117")
+      (reference "SW1") (unit 1) (value "SW_Push") (footprint "footprints:SW_Tactile_SPST_Angled_MJTP1117_fixed")
     )
     (path "/726b4788-4eb6-41d6-b1fb-ac076eabdb2c"
