File: case/pcb-case-complete.kicad_pcb (KiCad board)
At the start: 2 copper layers, 309.7 x 145.3 mm, 10 parts

Commit message: Updated casing plates.
Changed lines of the file:
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@@
       (layerselection 0x00010fc_ffffffff)
       (disableapertmacros false)
-      (usegerberextensions true)
+      (usegerberextensions false)
       (usegerberattributes false)
       (usegerberadvancedattributes false)
@@
       (plotinvisibletext false)
       (sketchpadsonfab false)
-      (subtractmaskfromsilk true)
+      (subtractmaskfromsilk false)
       (outputformat 1)
       (mirror false)
@@
       (effects (font (size 1.27 1.27) (thickness 0.15)))
     )
-    (pad "" thru_hole circle locked (at 0 0 90) (size 3 3) (drill 1.8) (layers *.Cu *.Mask "Dwgs.User")
+    (pad "" thru_hole circle locked (at 0 0 306) (size 3.2 3.2) (drill 2) (layers *.Cu *.Mask "Dwgs.User")
       (clearance 0.3))
   )
@@
       (effects (font (size 1.27 1.27) (thickness 0.15)))
     )
-    (pad "" thru_hole circle locked (at 0 0 90) (size 3 3) (drill 1.8) (layers *.Cu *.Mask "Dwgs.User")
+    (pad "" thru_hole circle locked (at 0 0 306) (size 3.2 3.2) (drill 2) (layers *.Cu *.Mask "Dwgs.User")
       (clearance 0.3))
   )
@@
       (effects (font (size 1.27 1.27) (thickness 0.15)))
     )
-    (pad "" thru_hole circle locked (at 0 0 90) (size 3 3) (drill 1.8) (layers *.Cu *.Mask "Dwgs.User")
+    (pad "" thru_hole circle locked (at 0 0 306) (size 3.2 3.2) (drill 2) (layers *.Cu *.Mask "Dwgs.User")
       (clearance 0.3))
   )
@@
       (effects (font (size 1.27 1.27) (thickness 0.15)))
     )
-    (pad "" thru_hole circle locked (at 0 0 90) (size 3 3) (drill 1.8) (layers *.Cu *.Mask "Dwgs.User")
+    (pad "" thru_hole circle locked (at 0 0 306) (size 3.2 3.2) (drill 2) (layers *.Cu *.Mask "Dwgs.User")
       (clearance 0.3))
   )
@@
       (effects (font (size 1.27 1.27) (thickness 0.15)))
     )
-    (pad "" thru_hole circle locked (at 0 0 90) (size 3 3) (drill 1.8) (layers *.Cu *.Mask "Dwgs.User")
+    (pad "" thru_hole circle locked (at 0 0 306) (size 3.2 3.2) (drill 2) (layers *.Cu *.Mask "Dwgs.User")
       (clearance 0.3))
   )
@@
       (effects (font (size 1.27 1.27) (thickness 0.15)) (justify mirror))
     )
-    (pad "" thru_hole circle locked (at 0 0 90) (size 3 3) (drill 1.8) (layers *.Cu *.Mask "Dwgs.User")
+    (pad "" thru_hole circle locked (at 0 0 90) (size 3.2 3.2) (drill 2) (layers *.Cu *.Mask "Dwgs.User")
       (clearance 0.3))
   )
@@
       (effects (font (size 1.27 1.27) (thickness 0.15)) (justify mirror))
     )
-    (pad "" thru_hole circle locked (at 0 0 90) (size 3 3) (drill 1.8) (layers *.Cu *.Mask "Dwgs.User")
+    (pad "" thru_hole circle locked (at 0 0 90) (size 3.2 3.2) (drill 2) (layers *.Cu *.Mask "Dwgs.User")
       (clearance 0.3))
   )
@@
       (effects (font (size 1.27 1.27) (thickness 0.15)) (justify mirror))
     )
-    (pad "" thru_hole circle locked (at 0 0 90) (size 3 3) (drill 1.8) (layers *.Cu *.Mask "Dwgs.User")
+    (pad "" thru_hole circle locked (at 0 0 90) (size 3.2 3.2) (drill 2) (layers *.Cu *.Mask "Dwgs.User")
       (clearance 0.3))
   )
@@
       (effects (font (size 1.27 1.27) (thickness 0.15)) (justify mirror))
     )
-    (pad "" thru_hole circle locked (at 0 0 90) (size 3 3) (drill 1.8) (layers *.Cu *.Mask "Dwgs.User")
+    (pad "" thru_hole circle locked (at 0 0 90) (size 3.2 3.2) (drill 2) (layers *.Cu *.Mask "Dwgs.User")
       (clearance 0.3))
   )
@@
       (effects (font (size 1.27 1.27) (thickness 0.15)) (justify mirror))
     )
-    (pad "" thru_hole circle locked (at 0 0 90) (size 3 3) (drill 1.8) (layers *.Cu *.Mask "Dwgs.User")
+    (pad "" thru_hole circle locked (at 0 0 90) (size 3.2 3.2) (drill 2) (layers *.Cu *.Mask "Dwgs.User")
       (clearance 0.3))
   )
