File: case/pcb-case.kicad_pcb (KiCad board)
At the start: 2 copper layers, 154.9 x 145.3 mm, 5 parts

Commit message: Updated casing plates.
Other:
- board text removed: "-14"
- board text removed: "14"
- board text removed: "60"
Changed lines of the file:
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@@
       (effects (font (size 1.27 1.27) (thickness 0.15)))
     )
-    (pad "" thru_hole circle locked (at 0 0 90) (size 3 3) (drill 1.8) (layers *.Cu *.Mask "Dwgs.User")
+    (pad "" thru_hole circle locked (at 0 0 90) (size 3.2 3.2) (drill 2) (layers *.Cu *.Mask "Dwgs.User")
       (clearance 0.3))
   )
@@
       (effects (font (size 1.27 1.27) (thickness 0.15)))
     )
-    (pad "" thru_hole circle locked (at 0 0 90) (size 3 3) (drill 1.8) (layers *.Cu *.Mask "Dwgs.User")
+    (pad "" thru_hole circle locked (at 0 0 90) (size 3.2 3.2) (drill 2) (layers *.Cu *.Mask "Dwgs.User")
       (clearance 0.3))
   )
@@
       (effects (font (size 1.27 1.27) (thickness 0.15)))
     )
-    (pad "" thru_hole circle locked (at 0 0 90) (size 3 3) (drill 1.8) (layers *.Cu *.Mask "Dwgs.User")
+    (pad "" thru_hole circle locked (at 0 0 90) (size 3.2 3.2) (drill 2) (layers *.Cu *.Mask "Dwgs.User")
       (clearance 0.3))
   )
@@
       (effects (font (size 1.27 1.27) (thickness 0.15)))
     )
-    (pad "" thru_hole circle locked (at 0 0 90) (size 3 3) (drill 1.8) (layers *.Cu *.Mask "Dwgs.User")
+    (pad "" thru_hole circle locked (at 0 0 90) (size 3.2 3.2) (drill 2) (layers *.Cu *.Mask "Dwgs.User")
       (clearance 0.3))
   )
@@
       (effects (font (size 1.27 1.27) (thickness 0.15)))
     )
-    (pad "" thru_hole circle locked (at 0 0 90) (size 3 3) (drill 1.8) (layers *.Cu *.Mask "Dwgs.User")
+    (pad "" thru_hole circle locked (at 0 0 90) (size 3.2 3.2) (drill 2) (layers *.Cu *.Mask "Dwgs.User")
       (clearance 0.3))
   )
@@
   (gr_line (start 251.22791 110.672541) (end 252.204501 124.638438) (layer "Edge.Cuts") (width 0.05))
   (gr_line (start 212.183237 96.174855) (end 198.868445 100.501095) (layer "Edge.Cuts") (width 0.05))
-  (gr_text "14" (at 251.891315 107.389862 18) (layer "Cmts.User")
-    (effects (font (size 1 1) (thickness 0.15)))
-  )
-  (gr_text "-14" (at 191.119955 127.242501 18) (layer "Cmts.User")
-    (effects (font (size 1 1) (thickness 0.15)))
-  )
-  (gr_text "60" (at 181.291248 128.967148 18) (layer "Cmts.User")
-    (effects (font (size 1 1) (thickness 0.15)))
-  )
   (zone locked (net 0) (net_name "") (layer "F.Cu") (hatch edge 0.508)
     (connect_pads (clearance 0.508))
