File: case/v2-choc/v2-choc-top.kicad_pcb (KiCad board)
At the start: 2 copper layers, 299.3 x 138.8 mm, 10 parts

Commit message: Removed copper layer from case, to make it thinner.
Routing:
- removed copper zone on B.Cu, net GND
- removed copper zone on F.Cu, net GND
Other:
- board text removed: "-14"
- board text removed: "60"
