File: case/v2-choc-basil/v2-choc-bottom.kicad_pcb (KiCad board)
At the start: 2 copper layers, 291.5 x 127.8 mm, 12 parts, among them SW1 SW_Push

Commit message: Fixed bottom case, added gerber files.
Parts:
- removed SW1: SW_Push, footprints:PushSwitch
Changed lines of the file:
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@@
       (clearance 0.3))
-  )
-  (footprint "footprints:PushSwitch" (layer "B.Cu")
-    (at 216.127512 123.813169 -90)
-    (descr "tactile push button, 6x6mm e.g. PTS645xx series, height=9.5mm")
-    (tags "tact sw push 6mm smd")
-    (property "Sheetfile" "v2-choc-basil.kicad_sch")
-    (property "Sheetname" "")
-    (attr smd)
-    (fp_text reference "SW1" (at 0 4 90) (layer "B.SilkS") hide
-      (effects (font (size 1 1) (thickness 0.15)) (justify mirror))
-    )
-    (fp_text value "SW_Push" (at 0 -4.15 90) (layer "B.Fab")
-      (effects (font (size 1 1) (thickness 0.15)) (justify mirror))
-    )
-    (fp_text user "${REFERENCE}" (at 0 4 90) (layer "B.Fab")
-      (effects (font (size 1 1) (thickness 0.15)) (justify mirror))
-    )
-    (fp_line (start -3 3) (end -3 -3) (layer "B.Fab") (width 0.1))
-    (fp_line (start 3 3) (end -3 3) (layer "B.Fab") (width 0.1))
-    (fp_line (start -3 -3) (end 3 -3) (layer "B.Fab") (width 0.1))
-    (fp_line (start 3 -3) (end 3 3) (layer "B.Fab") (width 0.1))
-    (fp_circle (center 0 0) (end 1 0) (layer "B.Fab") (width 0.1) (fill none))
-    (pad "1" smd rect (at 3.1 1.8 270) (size 1.8 1.3) (layers "B.Cu" "B.Paste" "B.Mask")
-      (pinfunction "1") (pintype "passive"))
-    (pad "1" smd rect (at -3.1 1.75 270) (size 1.8 1.3) (layers "B.Cu" "B.Paste" "B.Mask")
-      (pinfunction "1") (pintype "passive"))
-    (pad "2" smd rect (at -3.1 -1.7 270) (size 1.8 1.3) (layers "B.Cu" "B.Paste" "B.Mask")
-      (net 1 "GND") (pinfunction "2") (pintype "passive"))
-    (pad "2" smd rect (at 3 -1.7 270) (size 1.8 1.3) (layers "B.Cu" "B.Paste" "B.Mask")
-      (net 1 "GND") (pinfunction "2") (pintype "passive"))
-    (model "${KISYS3DMOD}/Button_Switch_SMD.3dshapes/SW_PUSH_6mm_H9.5mm.wrl"
-      (offset (xyz 0 0 0))
-      (scale (xyz 1 1 1))
-      (rotate (xyz 0 0 0))
-    )
   )
   (gr_arc (start 72.06872 138.177914) (mid 70.64826 136.928333) (end 70.506805 135.041762) (layer "Edge.Cuts") (width 0.1))
