File: case/v2/pcb-case-bottom.kicad_pcb (KiCad board)
At the start: 2 copper layers, 309.7 x 145.3 mm, 10 parts

Commit message: Release of Atrety V2 MX.
Parts:
- added ?: , , F.Cu at (194.1, 108.4)
- added ?: , , F.Cu at (228.1, 108.6)
Other:
- board text added: "Power"
- board text added: "Reset"
Changed lines of the file:
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@@
     (pad_to_mask_clearance 0)
     (aux_axis_origin 10.31875 10.31875)
-    (grid_origin 365.016716 133.193877)
+    (grid_origin 228.126819 108.629208)
     (pcbplotparams
       (layerselection 0x00010fc_ffffffff)
@@
       (clearance 0.3))
   )
+  (footprint "" (layer "F.Cu")
+    (at 194.08482 108.375207)
+    (fp_text reference "" (at 0 0) (layer "F.SilkS")
+      (effects (font (size 1.27 1.27) (thickness 0.15)))
+    )
+    (fp_text value "" (at 0 0) (layer "F.SilkS")
+      (effects (font (size 1.27 1.27) (thickness 0.15)))
+    )
+    (pad "" thru_hole oval locked (at 0 0 90) (size 10 6) (drill oval 9 5) (layers F&B.Cu *.Mask "Dwgs.User")
+      (clearance 0.3))
+  )
   (footprint "" locked (layer "F.Cu")
     (at 245.478828 139.407797 18)
@@
     )
     (pad "" thru_hole circle locked (at 0 0 108) (size 3.2 3.2) (drill 2) (layers *.Cu *.Mask "Dwgs.User")
+      (clearance 0.3))
+  )
+  (footprint "" (layer "F.Cu")
+    (at 228.126819 108.629208)
+    (fp_text reference "" (at 0 0) (layer "F.SilkS")
+      (effects (font (size 1.27 1.27) (thickness 0.15)))
+    )
+    (fp_text value "" (at 0 0) (layer "F.SilkS")
+      (effects (font (size 1.27 1.27) (thickness 0.15)))
+    )
+    (pad "" thru_hole circle locked (at 0 0 90) (size 4 4) (drill 3.5) (layers F&B.Cu *.Mask "Dwgs.User")
       (clearance 0.3))
   )
@@
   (gr_line (start 57.669445 129.203568) (end 64.752712 107.403517) (layer "Edge.Cuts") (width 0.1))
   (gr_line (start 263.876149 164.777232) (end 256.812225 172.562369) (layer "Edge.Cuts") (width 0.1))
+  (gr_text "Power" (at 194.08482 114.375207) (layer "B.SilkS")
+    (effects (font (size 1 1) (thickness 0.15)) (justify mirror))
+  )
+  (gr_text "Reset" (at 228.126819 111.829208) (layer "B.SilkS")
+    (effects (font (size 1 1) (thickness 0.15)) (justify mirror))
+  )
   (zone (net 1) (net_name "GND") (layers F&B.Cu) (hatch edge 0.508)
     (connect_pads (clearance 0.508))

Commit message: fixed small issues for the v2 case.
Routing:
- added copper zone on B.Cu, net (none)
- added copper zone on F.Cu, net (none)
- removed copper zone on B.Cu, net GND
- removed copper zone on F.Cu, net GND
Changed lines of the file:
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@@
       (layerselection 0x00010fc_ffffffff)
       (disableapertmacros false)
-      (usegerberextensions false)
+      (usegerberextensions true)
       (usegerberattributes false)
       (usegerberadvancedattributes false)
@@
       (psa4output false)
       (plotreference true)
-      (plotvalue true)
+      (plotvalue false)
       (plotinvisibletext false)
       (sketchpadsonfab false)
-      (subtractmaskfromsilk false)
+      (subtractmaskfromsilk true)
       (outputformat 1)
       (mirror false)
@@
   )
   (net 0 "")
-  (net 1 "GND")
   (footprint "" locked (layer "F.Cu")
     (at 319.760783 59.788673 18)
@@
     (effects (font (size 1 1) (thickness 0.15)) (justify mirror))
   )
-  (zone (net 1) (net_name "GND") (layers F&B.Cu) (hatch edge 0.508)
+  (zone (net 0) (net_name "") (layers F&B.Cu) (hatch edge 0.508)
     (connect_pads (clearance 0.508))
     (min_thickness 0.254) (filled_areas_thickness no)
